File: hw/watering/conductivity.kicad_sch (KiCad schematic)
At the start: 11 parts, among them J6 Conn_01x02_Pin, Q1 2N7002, U11 STI3508

Commit message: reduced pcb size
Changed lines of the file:
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@@
 			)
 		)
-		(pin "i_out" input
+		(pin "i_out" output
 			(at 176.53 129.54 0)
 			(effects
