File: hw/watering/solar.kicad_sch (KiCad schematic)
At the start: 23 parts, among them U2 DRV8220DSG, U5 STI3508

Commit message: updated inductors
Parts:
- removed L3, L4, L7: 22u, Inductor_SMD:L_Wuerth_MAPI-4030, symbol Device:L
- added L13, L14, L9: 22u, Inductor_SMD:L_Changjiang_FTC303020D, symbol Device:L
Connections:
- net V_bat: now also L9.1
- net current_meas/i_in: now also L14.2
- net current_meas1/i_out: now also L13.2
- net at D5.2 (A), U5.1 (LX): now also L9.2
- net at U2.2 (OUT1): now also L14.1
- net at U2.3 (OUT2): now also L13.1
