File: hw/watering/controller.kicad_sch (KiCad schematic)
At the start: 23 parts, among them SW2 KMS221GLFS, SW3 KMS221GLFS, U1 ESP32-C6, U3 W25Q128JVS, Y1 40MHz, Y2 32768Hz

Commit message: - hw   - rewired power input for battery   - some first placing of parts on pcb but no routing - sw   - added example http server from examples to server.cpp, not compilable yet
Parts:
- removed R33, R34: 47, Resistor_SMD:R_0603_1608Metric, symbol Device:R
Connections:
- net USBDM: now also U1.18 (GPIO12/USB_D-)
- net USBDP: now also U1.19 (GPIO13/USB_D+)
- net power-enable: now reaches U1.13 (MTDO/GPIO7/FSPID)
Other:
- moved on the sheet: AE1, C1, C2, C20, C22, C3, C4, R10, R14, R31, R32, R35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
