File: hw/watering/_restore_backup_2026-10-02T01-48-00-605/solar.kicad_sch (KiCad schematic)
At the start: 7 parts, among them U2 DRV8220DSG

Commit message: - sw   - charging batteries with solar somewhat works. mppt tracking is not possible because i messed up the current measurement   - implemented pid controller for current control. not operative, since current meas isn't working. maybe a voltage correlation is possibe? - hw   - current measurement is bad. output voltage of usb current is not high enough since input voltages are higher   - usb voltage wasn't connected correctly for charging   - solving by making battery voltage the main voltage bus on pcb and have all voltage users capped by switches to prevent battery drainage
Connections:
- net +5V: no longer C40.1, C41.1, C42.1, C43.1
- net current_meas/i_out: no longer L13.2
- net current_meas1/i_out: no longer L14.2
- net solar_pwm: now also U2.6 (IN1/PH); no longer U2.5 (IN2/EN)
- net usb_pwm: no longer U2.6 (IN1/PH)
- new net: C40.1, C41.1, C42.1, C43.1
Other:
- sheet bat ports: added none; removed +3V3
- moved on the sheet: C40, C41, C42, C43, L13, L14, U2
